File: eagle/rc2014_template.brd (EAGLE design)
At the start: 101.3 x 38.1 mm, 5 parts, among them IC1 74LS138N

Commit message: Fix wiring issue with template
Connections:
- net N$4: now also PIN1.10; no longer PIN1.8
- net N$5: now also PIN1.11; no longer PIN1.7
- net N$6: now also PIN1.12; no longer PIN1.6
Routing:
- net N$6: track 3.81 -> 23.0 mm
- net N$5: track 3.81 -> 16.8 mm
- net N$4: track 3.81 -> 10.1 mm
Changed lines of the file:
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@@
 <wire x1="21.59" y1="6.35" x2="21.59" y2="2.54" width="0.4064" layer="1"/>
-</signal>
-<signal name="N$4">
-<contactref element="PIN1" pad="8"/>
-<contactref element="IC1" pad="3"/>
-<wire x1="19.05" y1="6.35" x2="19.05" y2="2.54" width="0.4064" layer="1"/>
-</signal>
-<signal name="N$5">
-<contactref element="PIN1" pad="7"/>
-<contactref element="IC1" pad="2"/>
-<wire x1="16.51" y1="6.35" x2="16.51" y2="2.54" width="0.4064" layer="1"/>
-</signal>
-<signal name="N$6">
-<contactref element="PIN1" pad="6"/>
-<contactref element="IC1" pad="1"/>
-<wire x1="13.97" y1="6.35" x2="13.97" y2="2.54" width="0.4064" layer="1"/>
 </signal>
 <signal name="N$7">
@@
 <wire x1="31.75" y1="20.32" x2="29.21" y2="20.32" width="0" layer="19" extent="1-1"/>
 </signal>
+<signal name="N$4">
+<contactref element="PIN1" pad="10"/>
+<contactref element="IC1" pad="3"/>
+<wire x1="22.0318875" y1="8.0772" x2="22.86" y2="7.2490875" width="0.4064" layer="1"/>
+<wire x1="22.86" y1="7.2490875" x2="22.86" y2="3.81" width="0.4064" layer="1"/>
+<wire x1="22.86" y1="3.81" x2="24.13" y2="2.54" width="0.4064" layer="1"/>
+<wire x1="19.05" y1="6.35" x2="19.4209125" y2="6.35" width="0.4064" layer="1"/>
+<wire x1="19.4209125" y1="6.35" x2="21.1481125" y2="8.0772" width="0.4064" layer="1"/>
+<wire x1="21.1481125" y1="8.0772" x2="22.0318875" y2="8.0772" width="0.4064" layer="1"/>
+</signal>
+<signal name="N$5">
+<contactref element="PIN1" pad="11"/>
+<contactref element="IC1" pad="2"/>
+<wire x1="16.51" y1="6.35" x2="16.8809125" y2="6.35" width="0.4064" layer="1"/>
+<wire x1="25.1968" y1="8.6868" x2="25.4" y2="8.89" width="0.4064" layer="1"/>
+<wire x1="16.8809125" y1="6.35" x2="19.2177125" y2="8.6868" width="0.4064" layer="1"/>
+<wire x1="19.2177125" y1="8.6868" x2="25.1968" y2="8.6868" width="0.4064" layer="1"/>
+<wire x1="25.4" y1="8.89" x2="25.4" y2="3.81" width="0.4064" layer="1"/>
+<wire x1="25.4" y1="3.81" x2="26.67" y2="2.54" width="0.4064" layer="1"/>
+</signal>
+<signal name="N$6">
+<contactref element="PIN1" pad="12"/>
+<contactref element="IC1" pad="1"/>
+<wire x1="16.0681125" y1="8.0772" x2="16.9672" y2="8.0772" width="0.4064" layer="1"/>
+<wire x1="13.97" y1="6.35" x2="14.3409125" y2="6.35" width="0.4064" layer="1"/>
+<wire x1="14.3409125" y1="6.35" x2="16.0681125" y2="8.0772" width="0.4064" layer="1"/>
+<wire x1="19.05" y1="10.16" x2="26.67" y2="10.16" width="0.4064" layer="1"/>
+<wire x1="26.67" y1="10.16" x2="27.94" y2="8.89" width="0.4064" layer="1"/>
+<wire x1="27.94" y1="8.89" x2="27.94" y2="3.81" width="0.4064" layer="1"/>
+<wire x1="27.94" y1="3.81" x2="29.21" y2="2.54" width="0.4064" layer="1"/>
+<wire x1="16.9672" y1="8.0772" x2="19.05" y2="10.16" width="0.4064" layer="1"/>
+</signal>
 </signals>
