File: eagle/8085_board/rc2014_8085.brd (EAGLE design)
At the start: 101.3 x 50.8 mm, 17 parts, among them IC1 74HCT14N, IC3 74HCT573N

Commit message: Fixed wiring error on PCB
Parts:
- R3, R4: value 10K -> 1K
Connections:
- net N$2 renamed ALE
- net N$3 renamed TX
- net N$4 renamed RX
Routing:
- net GND: track 183.0 -> 220.3 mm
- net RESET: track 36.2 -> 47.9 mm
Other:
- board text added: "8085 CPU Board Designed for RC2014"
- board text added: "OPTIONAL"
- board text removed: "RC2014 8085 CPU Board"
Changed lines of the file:
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@@
 <?xml version="1.0" encoding="utf-8"?>
 <!DOCTYPE eagle SYSTEM "eagle.dtd">
-<eagle version="8.1.0">
+<eagle version="8.1.1">
 <drawing>
 <settings>
@@
 <wire x1="101.27" y1="50.79" x2="0" y2="50.79" width="0" layer="20"/>
 <wire x1="0" y1="0" x2="0" y2="50.79" width="0" layer="20"/>
-<text x="97.155" y="19.05" size="1.27" layer="25" rot="R90">ancientcomputing</text>
-<text x="94.615" y="19.05" size="1.9304" layer="25" rot="R90">RC2014 8085 CPU Board</text>
+<text x="7.62" y="8.89" size="1.27" layer="25">ancientcomputing</text>
+<text x="7.62" y="19.05" size="1.778" layer="25">8085 CPU Board
+Designed for RC2014</text>
 <text x="71.755" y="32.385" size="2.1844" layer="25">8085</text>
 <text x="83.185" y="14.605" size="1.778" layer="25">'573</text>
 <text x="18.415" y="34.925" size="1.778" layer="25">'14</text>
+<text x="56.515" y="12.7" size="1.27" layer="25" rot="R90">OPTIONAL</text>
 </plain>
 <attributes>
@@
 <element name="C2" library="rcl" package="C050-024X044" value="0.1uF" x="52.07" y="17.78" rot="R90"/>
 <element name="R2" library="rcl" package="0207/10" value="10K" x="7.62" y="27.305"/>
-<element name="R3" library="rcl" package="0207/10" value="10K" x="78.74" y="45.72"/>
-<element name="R4" library="rcl" package="0207/10" value="10K" x="78.74" y="48.26"/>
+<element name="R3" library="rcl" package="0207/10" value="1K" x="78.74" y="45.72"/>
+<element name="R4" library="rcl" package="0207/10" value="1K" x="78.74" y="48.26"/>
 </elements>
 <signals>
@@
 <wire x1="43.18" y1="40.64" x2="43.18" y2="47.625" width="0.4064" layer="1"/>
 <wire x1="43.18" y1="47.625" x2="42.545" y2="48.26" width="0.4064" layer="1"/>
-<wire x1="42.545" y1="48.26" x2="40.64" y2="48.26" width="0.4064" layer="1"/>
+<wire x1="41.275" y1="48.26" x2="42.545" y2="48.26" width="0.4064" layer="1"/>
+<wire x1="41.275" y1="48.26" x2="40.64" y2="48.26" width="0.4064" layer="1"/>
 <wire x1="53.34" y1="25.4" x2="53.34" y2="22.225" width="0.4064" layer="16"/>
 <wire x1="55.88" y1="22.225" x2="58.42" y2="22.225" width="0.4064" layer="16"/>
@@
 <wire x1="36.83" y1="15.875" x2="34.925" y2="17.78" width="0.8128" layer="1"/>
 <wire x1="34.925" y1="17.78" x2="34.925" y2="29.845" width="0.8128" layer="1"/>
-<wire x1="34.925" y1="29.845" x2="33.02" y2="31.75" width="0.8128" layer="1"/>
-<wire x1="33.02" y1="31.75" x2="22.86" y2="31.75" width="0.8128" layer="1"/>
+<wire x1="34.925" y1="29.845" x2="33.3375" y2="31.4325" width="0.8128" layer="1"/>
+<wire x1="33.3375" y1="31.4325" x2="33.02" y2="31.75" width="0.8128" layer="1"/>
+<wire x1="22.86" y1="31.75" x2="33.02" y2="31.75" width="0.8128" layer="1"/>
 <wire x1="66.04" y1="21.59" x2="92.71" y2="21.59" width="0.4064" layer="16"/>
-<wire x1="20.32" y1="39.37" x2="15.24" y2="43.18" width="0" layer="19" extent="1-1"/>
+<wire x1="15.24" y1="43.18" x2="19.685" y2="43.18" width="0.4064" layer="1"/>
+<wire x1="19.685" y1="43.18" x2="20.32" y2="42.545" width="0.4064" layer="1"/>
+<wire x1="20.32" y1="42.545" x2="20.32" y2="39.37" width="0.4064" layer="1"/>
+<wire x1="20.32" y1="39.37" x2="20.32" y2="36.83" width="0.4064" layer="1"/>
+<wire x1="22.86" y1="34.29" x2="22.86" y2="31.75" width="0.4064" layer="1"/>
+<wire x1="20.32" y1="36.83" x2="22.86" y2="34.29" width="0.4064" layer="1"/>
+<wire x1="33.3375" y1="31.4325" x2="33.3375" y2="40.3225" width="0.4064" layer="1"/>
+<wire x1="33.3375" y1="40.3225" x2="41.275" y2="48.26" width="0.4064" layer="1"/>
+<wire x1="53.34" y1="22.225" x2="52.07" y2="15.24" width="0" layer="19" extent="16-16"/>
+<wire x1="40.64" y1="15.875" x2="41.275" y2="15.24" width="0" layer="19" extent="1-1"/>
+<wire x1="17.78" y1="31.75" x2="22.86" y2="31.75" width="0" layer="19" extent="1-1"/>
+<wire x1="2.54" y1="34.29" x2="1.8288" y2="43.4594" width="0" layer="19" extent="1-1"/>
 </signal>
 <signal name="VCC">
@@
 <wire x1="17.78" y1="49.53" x2="31.75" y2="49.53" width="0.4064" layer="16"/>
 <wire x1="31.75" y1="49.53" x2="33.02" y2="48.26" width="0.4064" layer="16"/>
-<wire x1="8.3312" y1="47.9806" x2="10.16" y2="39.37" width="0" layer="19" extent="1-1"/>
+<wire x1="15.24" y1="48.26" x2="13.97" y2="48.26" width="0.4064" layer="1"/>
+<wire x1="13.97" y1="48.26" x2="11.43" y2="45.72" width="0.4064" layer="1"/>
+<wire x1="11.43" y1="45.72" x2="11.43" y2="42.545" width="0.4064" layer="1"/>
+<wire x1="11.43" y1="42.545" x2="10.16" y2="41.275" width="0.4064" layer="1"/>
+<wire x1="10.16" y1="41.275" x2="10.16" y2="39.37" width="0.4064" layer="1"/>
 </signal>
 <signal name="N$15">
@@
 <wire x1="60.96" y1="37.465" x2="60.96" y2="40.64" width="0.4064" layer="1"/>
 </signal>
-<signal name="N$2">
+<signal name="ALE">
 <contactref element="IC3" pad="11"/>
 <contactref element="IC2" pad="30"/>
@@
 <wire x1="11.43" y1="34.925" x2="55.245" y2="34.925" width="0.4064" layer="16"/>
 </signal>
-<signal name="N$3">
+<signal name="TX">
 <contactref element="R4" pad="1"/>
 <contactref element="FTDIGND" pad="5"/>
@@
 <wire x1="71.755" y1="48.26" x2="69.215" y2="45.72" width="0.4064" layer="1"/>
 </signal>
-<signal name="N$4">
+<signal name="RX">
 <contactref element="R3" pad="1"/>
 <contactref element="FTDIGND" pad="4"/>
@@
 </board>
 </drawing>
+<compatibility>
+<note version="6.3" minversion="6.2.2" severity="warning">
+Since Version 6.2.2 text objects can contain more than one line,
+which will not be processed correctly with this version.
+</note>
+</compatibility>
 </eagle>

Commit message: Clean up, add CLK
Connections:
- net CLK: now also IC2.37
Routing:
- net CLK: track 0.00 -> 44.2 mm, vias 0 -> 2
- net GND: track 220.3 -> 248.0 mm
- net RESET: track 47.9 -> 55.8 mm, vias 0 -> 1
- net VCC: track 201.7 -> 203.2 mm
- net A1: track 41.9 -> 43.2 mm
Other:
- board text added: "1K"
Changed lines of the file:
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@@
 <text x="18.415" y="34.925" size="1.778" layer="25">'14</text>
 <text x="56.515" y="12.7" size="1.27" layer="25" rot="R90">OPTIONAL</text>
+<text x="85.09" y="46.355" size="1.778" layer="25">1K</text>
 </plain>
 <attributes>
@@
 <contactref element="IC1" pad="7"/>
 <contactref element="S1" pad="3"/>
-<wire x1="1.8288" y1="43.4594" x2="8.3312" y2="43.4594" width="0.4064" layer="16"/>
+<wire x1="8.3312" y1="43.4594" x2="1.8288" y2="43.4594" width="0.4064" layer="1"/>
 <wire x1="8.3312" y1="43.4594" x2="12.4206" y2="43.4594" width="0.4064" layer="16"/>
 <wire x1="12.4206" y1="43.4594" x2="12.7" y2="43.18" width="0.4064" layer="16"/>
@@
 <contactref element="IC2" pad="39"/>
 <contactref element="FTDIGND" pad="1"/>
-<via x="41.275" y="15.24" extent="1-16" drill="0.6096"/>
-<wire x1="41.275" y1="15.24" x2="60.325" y2="15.24" width="0.6096" layer="16"/>
+<via x="41.91" y="15.24" extent="1-16" drill="0.6096"/>
+<wire x1="52.07" y1="15.24" x2="41.91" y2="15.24" width="0.6096" layer="16"/>
+<wire x1="52.07" y1="15.24" x2="60.325" y2="15.24" width="0.6096" layer="16"/>
 <wire x1="60.325" y1="15.24" x2="64.135" y2="19.05" width="0.6096" layer="16"/>
 <wire x1="64.135" y1="19.05" x2="66.04" y2="19.05" width="0.6096" layer="16"/>
@@
 <wire x1="66.04" y1="19.05" x2="66.04" y2="21.59" width="0.4064" layer="16"/>
 <contactref element="C2" pad="1"/>
-<wire x1="41.91" y1="2.54" x2="41.91" y2="14.605" width="0.8128" layer="1"/>
-<wire x1="41.91" y1="14.605" x2="40.64" y2="15.875" width="0.8128" layer="1"/>
-<wire x1="40.64" y1="15.875" x2="36.83" y2="15.875" width="0.8128" layer="1"/>
-<wire x1="36.83" y1="15.875" x2="34.925" y2="17.78" width="0.8128" layer="1"/>
+<wire x1="41.91" y1="2.54" x2="41.91" y2="15.24" width="0.8128" layer="1"/>
+<wire x1="41.91" y1="15.24" x2="37.465" y2="15.24" width="0.8128" layer="1"/>
+<wire x1="37.465" y1="15.24" x2="34.925" y2="17.78" width="0.8128" layer="1"/>
 <wire x1="34.925" y1="17.78" x2="34.925" y2="29.845" width="0.8128" layer="1"/>
 <wire x1="34.925" y1="29.845" x2="33.3375" y2="31.4325" width="0.8128" layer="1"/>
@@
 <wire x1="22.86" y1="31.75" x2="33.02" y2="31.75" width="0.8128" layer="1"/>
 <wire x1="66.04" y1="21.59" x2="92.71" y2="21.59" width="0.4064" layer="16"/>
-<wire x1="15.24" y1="43.18" x2="19.685" y2="43.18" width="0.4064" layer="1"/>
-<wire x1="19.685" y1="43.18" x2="20.32" y2="42.545" width="0.4064" layer="1"/>
-<wire x1="20.32" y1="42.545" x2="20.32" y2="39.37" width="0.4064" layer="1"/>
 <wire x1="20.32" y1="39.37" x2="20.32" y2="36.83" width="0.4064" layer="1"/>
 <wire x1="22.86" y1="34.29" x2="22.86" y2="31.75" width="0.4064" layer="1"/>
@@
 <wire x1="33.3375" y1="31.4325" x2="33.3375" y2="40.3225" width="0.4064" layer="1"/>
 <wire x1="33.3375" y1="40.3225" x2="41.275" y2="48.26" width="0.4064" layer="1"/>
-<wire x1="53.34" y1="22.225" x2="52.07" y2="15.24" width="0" layer="19" extent="16-16"/>
-<wire x1="40.64" y1="15.875" x2="41.275" y2="15.24" width="0" layer="19" extent="1-1"/>
-<wire x1="17.78" y1="31.75" x2="22.86" y2="31.75" width="0" layer="19" extent="1-1"/>
-<wire x1="2.54" y1="34.29" x2="1.8288" y2="43.4594" width="0" layer="19" extent="1-1"/>
+<wire x1="15.24" y1="43.18" x2="19.685" y2="43.18" width="0.4064" layer="16"/>
+<wire x1="19.685" y1="43.18" x2="20.32" y2="42.545" width="0.4064" layer="16"/>
+<wire x1="20.32" y1="42.545" x2="20.32" y2="39.37" width="0.4064" layer="16"/>
+<wire x1="1.8288" y1="43.4594" x2="1.8288" y2="42.4688" width="0.4064" layer="1"/>
+<wire x1="1.8288" y1="42.4688" x2="1.2192" y2="41.8592" width="0.4064" layer="1"/>
+<wire x1="1.2192" y1="41.8592" x2="1.2192" y2="34.9758" width="0.4064" layer="1"/>
+<wire x1="1.905" y1="34.29" x2="2.54" y2="34.29" width="0.4064" layer="1"/>
+<wire x1="1.2192" y1="34.9758" x2="1.905" y2="34.29" width="0.4064" layer="1"/>
+<wire x1="53.34" y1="22.225" x2="53.34" y2="16.51" width="0.4064" layer="16"/>
+<wire x1="53.34" y1="16.51" x2="52.07" y2="15.24" width="0.4064" layer="16"/>
+<wire x1="17.78" y1="31.75" x2="17.78" y2="29.21" width="0.4064" layer="16"/>
+<wire x1="17.78" y1="29.21" x2="22.86" y2="29.21" width="0.4064" layer="16"/>
+<wire x1="22.86" y1="29.21" x2="22.86" y2="31.75" width="0.4064" layer="16"/>
 </signal>
 <signal name="VCC">
@@
 <contactref element="IC2" pad="35"/>
 <wire x1="7.62" y1="39.37" x2="7.62" y2="40.005" width="0.6096" layer="16"/>
-<wire x1="7.62" y1="40.005" x2="8.89" y2="41.275" width="0.6096" layer="16"/>
-<wire x1="8.89" y1="41.275" x2="21.59" y2="41.275" width="0.6096" layer="16"/>
-<wire x1="21.59" y1="41.275" x2="22.86" y2="42.545" width="0.6096" layer="16"/>
 <wire x1="40.64" y1="40.64" x2="40.64" y2="43.18" width="0.6096" layer="1"/>
 <wire x1="53.34" y1="43.18" x2="40.64" y2="43.18" width="0.6096" layer="16"/>
@@
 <wire x1="36.195" y1="38.1" x2="38.735" y2="40.64" width="0.8128" layer="1"/>
 <wire x1="38.735" y1="40.64" x2="40.64" y2="40.64" width="0.8128" layer="1"/>
+<wire x1="7.62" y1="39.37" x2="7.62" y2="40.005" width="0.6096" layer="1"/>
+<wire x1="7.62" y1="40.005" x2="8.89" y2="41.275" width="0.6096" layer="1"/>
+<wire x1="8.89" y1="41.275" x2="19.685" y2="41.275" width="0.6096" layer="1"/>
+<wire x1="19.685" y1="41.275" x2="22.86" y2="44.45" width="0.6096" layer="1"/>
 </signal>
 <signal name="A7">
@@
 <wire x1="36.83" y1="6.35" x2="71.12" y2="6.35" width="0.4064" layer="16"/>
 <via x="71.12" y="6.35" extent="1-16" drill="0.6096"/>
-<wire x1="71.12" y1="6.35" x2="71.12" y2="10.16" width="0.4064" layer="1"/>
+<wire x1="71.12" y1="6.35" x2="71.12" y2="11.43" width="0.4064" layer="1"/>
 <wire x1="36.83" y1="2.54" x2="36.83" y2="6.35" width="0.4064" layer="16"/>
-<wire x1="71.12" y1="10.16" x2="71.12" y2="11.43" width="0" layer="19" extent="1-1"/>
 </signal>
 <signal name="A2">
@@
 <signal name="CLK">
 <contactref element="_PIN1" pad="21"/>
+<contactref element="IC2" pad="37"/>
+<wire x1="48.26" y1="40.64" x2="48.26" y2="38.735" width="0.4064" layer="1"/>
+<wire x1="48.26" y1="38.735" x2="46.99" y2="37.465" width="0.4064" layer="1"/>
+<wire x1="46.99" y1="37.465" x2="46.99" y2="24.13" width="0.4064" layer="1"/>
+<wire x1="46.99" y1="24.13" x2="48.26" y2="22.86" width="0.4064" layer="1"/>
+<via x="48.26" y="22.86" extent="1-16" drill="0.6096"/>
+<wire x1="48.26" y1="22.86" x2="50.8" y2="22.86" width="0.4064" layer="16"/>
+<via x="50.8" y="22.86" extent="1-16" drill="0.6096"/>
+<wire x1="50.8" y1="22.86" x2="51.435" y2="22.86" width="0.4064" layer="1"/>
+<wire x1="51.435" y1="22.86" x2="53.975" y2="20.32" width="0.4064" layer="1"/>
+<wire x1="53.975" y1="20.32" x2="53.975" y2="6.985" width="0.4064" layer="1"/>
+<wire x1="53.975" y1="6.985" x2="52.07" y2="5.08" width="0.4064" layer="1"/>
+<wire x1="52.07" y1="5.08" x2="52.07" y2="2.54" width="0.4064" layer="1"/>
 </signal>
 <signal name="/MREQ">
@@
 <contactref element="D1" pad="A"/>
 <contactref element="S1" pad="1"/>
-<wire x1="8.6106" y1="48.26" x2="15.24" y2="48.26" width="0.4064" layer="16"/>
+<wire x1="8.6106" y1="48.26" x2="15.24" y2="48.26" width="0.4064" layer="1"/>
 <wire x1="8.6106" y1="48.26" x2="8.3312" y2="47.9806" width="0.4064" layer="16"/>
-<wire x1="8.3312" y1="47.9806" x2="1.8288" y2="47.9806" width="0.4064" layer="16"/>
-<wire x1="33.02" y1="44.45" x2="33.02" y2="48.26" width="0.4064" layer="16"/>
-<wire x1="15.24" y1="48.26" x2="16.51" y2="48.26" width="0.4064" layer="16"/>
-<wire x1="16.51" y1="48.26" x2="17.78" y2="49.53" width="0.4064" layer="16"/>
-<wire x1="17.78" y1="49.53" x2="31.75" y2="49.53" width="0.4064" layer="16"/>
-<wire x1="31.75" y1="49.53" x2="33.02" y2="48.26" width="0.4064" layer="16"/>
-<wire x1="15.24" y1="48.26" x2="13.97" y2="48.26" width="0.4064" layer="1"/>
-<wire x1="13.97" y1="48.26" x2="11.43" y2="45.72" width="0.4064" layer="1"/>
-<wire x1="11.43" y1="45.72" x2="11.43" y2="42.545" width="0.4064" layer="1"/>
-<wire x1="11.43" y1="42.545" x2="10.16" y2="41.275" width="0.4064" layer="1"/>
-<wire x1="10.16" y1="41.275" x2="10.16" y2="39.37" width="0.4064" layer="1"/>
+<wire x1="8.3312" y1="47.9806" x2="1.8288" y2="47.9806" width="0.4064" layer="1"/>
+<via x="8.6106" y="48.26" extent="1-16" drill="0.6096"/>
+<wire x1="15.24" y1="48.26" x2="16.51" y2="48.26" width="0.4064" layer="1"/>
+<wire x1="16.51" y1="48.26" x2="17.78" y2="49.53" width="0.4064" layer="1"/>
+<wire x1="17.78" y1="49.53" x2="31.75" y2="49.53" width="0.4064" layer="1"/>
+<wire x1="31.75" y1="49.53" x2="33.02" y2="48.26" width="0.4064" layer="1"/>
+<wire x1="33.02" y1="48.26" x2="33.02" y2="44.45" width="0.4064" layer="1"/>
+<wire x1="8.3312" y1="47.9806" x2="6.7056" y2="47.9806" width="0.4064" layer="16"/>
+<wire x1="6.7056" y1="47.9806" x2="5.08" y2="46.355" width="0.4064" layer="16"/>
+<wire x1="5.08" y1="38.735" x2="6.985" y2="36.83" width="0.4064" layer="16"/>
+<wire x1="9.525" y1="36.83" x2="10.16" y2="37.465" width="0.4064" layer="16"/>
+<wire x1="10.16" y1="37.465" x2="10.16" y2="39.37" width="0.4064" layer="16"/>
+<wire x1="5.08" y1="46.355" x2="5.08" y2="38.735" width="0.4064" layer="16"/>
+<wire x1="6.985" y1="36.83" x2="9.525" y2="36.83" width="0.4064" layer="16"/>
 </signal>
 <signal name="N$15">
