File: eagle/rr3kram/rc2014_3kb_ram.sch (EAGLE design)
At the start: 17 parts, among them IC7 74LS138N

Commit message: Fix missing A1, A0 lines
Connections:
- net N$1 renamed /RD
- new net /INT: _PIN1.22
- new net /RST: _PIN1.20
- new net CLK: _PIN1.21
- net A0: now also _PIN1.16
- net A1: now also _PIN1.15
