File: eagle/16550_board_rev_b/rc2014_16550b.sch (EAGLE design)
At the start: 13 parts, among them IC1 16C550, IC2 74HCT00N

Commit message: Correctly identify 74LS03
Parts:
- IC2: value 74HCT00N -> 74HCT03N
- R1, R2, R3: value (none) -> 4.7K
Changed lines of the file:
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@@
 <part name="GND4" library="supply1" deviceset="GND" device=""/>
 <part name="C4" library="rcl" deviceset="C-EU" device="050-024X044" value="0.1uF"/>
-<part name="IC2" library="74xx-eu" deviceset="74*00" device="N" technology="HCT"/>
-<part name="R1" library="rcl" deviceset="R-US_" device="0207/10"/>
-<part name="R2" library="rcl" deviceset="R-US_" device="0207/10"/>
-<part name="R3" library="rcl" deviceset="R-US_" device="0207/10"/>
+<part name="IC2" library="74xx-eu" deviceset="74*00" device="N" technology="HCT" value="74HCT03N"/>
+<part name="R1" library="rcl" deviceset="R-US_" device="0207/10" value="4.7K"/>
+<part name="R2" library="rcl" deviceset="R-US_" device="0207/10" value="4.7K"/>
+<part name="R3" library="rcl" deviceset="R-US_" device="0207/10" value="4.7K"/>
 <part name="P+4" library="supply1" deviceset="VCC" device=""/>
 <part name="JP1" library="pinhead" deviceset="PINHD-1X3" device=""/>
